Commit message: Fix xacro file path in launch file and update URDF mesh references for Pingu robot

File: Mujoco/pingu_mujoco_sim/description/urdf/pingu.urdf (robot description, URDF)
Before this commit: robot pingu, 12 links, 10 joints
Links:
- link base_link: geometry collision mesh filename=package://pingu_description/mesh/base_link.stl scale=1 1 1; visual mesh filename=package://pingu_description/mesh/base_link.stl scale=1 1 1

Commit message: Update controller configurations and fix joint names in URDF for Pingu robot

File: Mujoco/pingu_mujoco_sim/description/urdf/pingu.urdf (robot description, URDF)
Before this commit: robot pingu, 12 links, 10 joints
Joints:
- added joint rw_base_joint: type fixed, parent base_link, child rw_base, origin xyz=0 0 .2875 rpy=0 0 0
- joint base_joint: child rw_base -> base_link; parent base_link -> world; type fixed -> floating
